Commit message: feat & fix: resolve URDF LiDAR occlusion, update setup.py, and add yolo_vision_node for Tasks 1-4

File: urdf/my_robot_rgbd.urdf (robot description, URDF)
Before this commit: robot turtlebot3_burger, 9 links, 8 joints
Links:
- link my_rgbd_camera_link: geometry visual box size=0.02 0.05 0.02
